File: USBCWrover/USBCWrover kopie.kicad_pcb (KiCad board)
At the start: 2 copper layers, 31.5 x 42 mm, 18 parts, among them J1 USB_C_Receptacle_USB2.0, J2 Conn_02x10_Odd_Even, J3 Conn_02x10_Odd_Even, SW1 SW_Push, U1 UMH3N, U2 CP2104, U3 AMS1117-3.3, U4 ESP32-WROVER

Commit message: lot prettier
Parts:
- U3: value AMS1117-3.3 -> HX9193-33GB; footprint Package_TO_SOT_SMD:SOT-223-3_TabPin2 -> Package_TO_SOT_SMD:SOT-23-5
- moved U3 8.42 mm to (150.9, 133.9), turned to 180 degrees
- moved C6 8.36 mm to (145.9, 132.1), turned to 90 degrees
- moved C7 7.46 mm to (147.8, 132.1), turned to 90 degrees
- moved C4 4.66 mm to (154.7, 135.0)
- moved C5 4.55 mm to (154.7, 132.8)
- moved R5 4.10 mm to (132.2, 133.6), turned to 90 degrees
- moved U1 3.42 mm to (129.3, 133.7)
- moved R6 2.78 mm to (126.4, 133.6), turned to 90 degrees
- moved C1 2.75 mm to (144.0, 132.1), turned to 90 degrees
- moved U2 2.17 mm to (140.0, 133.2)
- moved C2 2.15 mm to (134.9, 132.6)
- moved R1 2.12 mm to (134.9, 135.1)
- moved J1 1.93 mm to (141.1, 142.5)
- moved R2 1.84 mm to (144.8, 135.1)
- moved SW1 1.53 mm to (130.6, 140.8)
Connections:
- J2 pad 10: Net-(J2-Pad10) -> IO17
- J2 pad 12: Net-(J2-Pad12) -> IO16
- U3 pad 1: GND -> +5V
- U3 pad 2: +3V3 -> GND
- U4 pad 27: Net-(U4-Pad27) -> IO16
- U4 pad 28: Net-(U4-Pad28) -> IO17
Routing:
- net GND: track 20.1 -> 64.0 mm, vias 23 -> 16
- net +3V3: track 90.0 -> 78.5 mm, vias 4 -> 5
- net SER_RTS: track 9.71 -> 16.0 mm
- net IO18: track 29.6 -> 24.5 mm
- net IO17: track 0.00 -> 3.17 mm
- net ESP_RST: track 53.7 -> 50.8 mm
- net IO16: track 0.00 -> 2.64 mm
- net USB_D+: track 7.76 -> 10.3 mm
- net IO23: track 27.6 -> 25.5 mm
- net ESP_RXD: track 40.1 -> 38.2 mm
- net SER_DTR: track 9.73 -> 11.6 mm
- net ESP_FLS: track 34.9 -> 36.7 mm
- net ESP_TXD: track 35.0 -> 36.6 mm
- net Net-(J1-PadB5): track 5.19 -> 3.80 mm
- net +5V: track 41.4 -> 40.6 mm, vias 4 -> 0
Other:
- board size 31.5 x 42 mm -> 31.5 x 40.5 mm
- board text added: "GND IO27 IO25 IO32 TDI IO4 IO0 IO2 SD1 CLK"
- board text added: "GND NC SVN IO35 IO33 IO34 TMS NC SD2 CMD"
- board text added: "JLCJLCJLCJLC"
- board text added: "RST SVP IO26 IO18 IO19 IO23 IO5 3.3v TCK SD3"
- board text added: "Reset"
- board text added: "TXD RXD IO22 IO21 IO17* IO16* GND 5V TDD SD0"
- board text added: "Wroom / Wrover"
- board text added: "https://git.io/JJAKG"
